Commit message: Make hande URDF compatible with other grippers

File: robotiq_description/urdf/robotiq_hande_macro.urdf.xacro (robot description, xacro)
@@ -41,5 +41,5 @@
     <!--  + Height added by the coupler: 13.9mm -->
     <!--  + Reference frame: at the middle (6.95mm) -->
-    <joint name="robotiq_coupler_joint" type="fixed">
+    <!-- <joint name="${prefix}robotiq_coupler_joint" type="fixed">
       <origin xyz="0 0 0.00695" rpy="0 0 ${-pi/2.0}" />
       <parent link="${parent}"/>
@@ -66,11 +66,12 @@
         <material name="DarkGrey" />
       </visual>
-    </link>
-    <joint name="${prefix}robotiq_hande_base_joint" type="fixed">
-      <origin rpy="0 0 0" xyz="0 0 0.055"/>
-      <parent link="${prefix}robotiq_coupler"/>
-      <child link="${prefix}hande_link"/>
+    </link> -->
+    <joint name="${prefix}hande_base_joint" type="fixed">
+      <!-- <origin rpy="0 0 0" xyz="0 0 0.055"/> -->
+      <parent link="${parent}"/>
+      <child link="${prefix}hande_base_link"/>
+      <xacro:insert_block name="origin" />
     </joint>
-    <link name="${prefix}hande_link">
+    <link name="${prefix}hande_base_link">
       <inertial>
         <mass value="0.86387"/>
@@ -96,5 +97,5 @@
     <joint name="${prefix}hande_left_finger_joint" type="prismatic">
       <origin rpy="0 0 0" xyz="0 -0.025 0.0345"/>
-      <parent link="${prefix}hande_link"/>
+      <parent link="${prefix}hande_base_link"/>
       <child link="${prefix}hande_left_finger"/>
       <axis xyz="0 1 0"/>
@@ -127,5 +128,5 @@
     <joint name="${prefix}hande_right_finger_joint" type="prismatic">
       <origin rpy="0 0 0" xyz="0 0.025 0.0345"/>
-      <parent link="${prefix}hande_link"/>
+      <parent link="${prefix}hande_base_link"/>
       <child link="${prefix}hande_right_finger"/>
       <axis xyz="0 -1 0"/>
@@ -159,5 +160,5 @@
     <joint name="${prefix}robotiq_hande_end_joint" type="fixed">
       <origin rpy="0 0 0" xyz="0 0 0.095"/>
-      <parent link="${prefix}hande_link"/>
+      <parent link="${prefix}hande_base_link"/>
       <child link="${prefix}hande_end"/>
     </joint>

Commit message: Fix gripper action direction difference between rviz and real situation

File: robotiq_description/urdf/robotiq_hande_macro.urdf.xacro (robot description, xacro)
@@ -96,8 +96,8 @@
     </link>
     <joint name="${prefix}hande_left_finger_joint" type="prismatic">
-      <origin rpy="0 0 0" xyz="0 -0.025 0.0345"/>
+      <origin rpy="0 0 0" xyz="0 -0.00025 0.0345"/>
       <parent link="${prefix}hande_base_link"/>
       <child link="${prefix}hande_left_finger"/>
-      <axis xyz="0 1 0"/>
+      <axis xyz="0 -1 0"/>
       <limit effort="130" lower="0" upper="0.025" velocity="0.15"/>
     </joint>
@@ -127,8 +127,8 @@
     </link>
     <joint name="${prefix}hande_right_finger_joint" type="prismatic">
-      <origin rpy="0 0 0" xyz="0 0.025 0.0345"/>
+      <origin rpy="0 0 0" xyz="0 0.00025 0.0345"/>
       <parent link="${prefix}hande_base_link"/>
       <child link="${prefix}hande_right_finger"/>
-      <axis xyz="0 -1 0"/>
+      <axis xyz="0 1 0"/>
       <limit effort="130" lower="0" upper="0.025" velocity="0.15"/>
       <mimic joint="${prefix}hande_left_finger_joint" multiplier="1" offset="0"/>

Commit message: remove some left overs

File: robotiq_description/urdf/robotiq_hande_macro.urdf.xacro (robot description, xacro)
@@ -96,5 +96,5 @@
     </link>
     <joint name="${prefix}hande_left_finger_joint" type="prismatic">
-      <origin rpy="0 0 0" xyz="0 -0.00025 0.0345"/>
+      <origin rpy="0 0 0" xyz="0 0 0.0345"/>
       <parent link="${prefix}hande_base_link"/>
       <child link="${prefix}hande_left_finger"/>
@@ -127,5 +127,5 @@
     </link>
     <joint name="${prefix}hande_right_finger_joint" type="prismatic">
-      <origin rpy="0 0 0" xyz="0 0.00025 0.0345"/>
+      <origin rpy="0 0 0" xyz="0 0 0.0345"/>
       <parent link="${prefix}hande_base_link"/>
       <child link="${prefix}hande_right_finger"/>
